Commit message: Pandora task now runs, need to make it not crash!

File: resources/robots/pandora/urdf/pandora_v1_robot.urdf (robot description, URDF)
Before this commit: robot pandora_v1, 13 links, 12 joints
Links:
- link l_ankle: geometry visual cylinder length=0.04 radius=0.015; visual mesh filename=../meshes/full_build_STL/Legs_Ankle_CrossGimbal2.stl scale=0.001 0.001 0.001
- link l_foot: geometry collision box size=0.2 0.10 0.03; visual cylinder length=0.04 radius=0.015
- link l_glute: geometry visual cylinder length=0.04 radius=0.015; visual mesh filename=../meshes/full_build_STL/Thigh_Top_Left_Ass.stl scale=0.001 0.001 0.001
- link l_hipgimbal: geometry visual cylinder length=0.04 radius=0.015; visual mesh filename=../meshes/full_build_STL/Cross_Gimble.stl scale=0.001 0.001 0.001
- link l_shin: geometry visual cylinder length=0.04 radius=0.015; visual mesh filename=../meshes/full_build_STL/Left_Shin_Assembly.stl scale=0.001 0.001 0.001
- link l_thigh: geometry visual cylinder length=0.04 radius=0.015; visual mesh filename=../meshes/full_build_STL/Thigh_Left_Assembly.stl scale=0.001 0.001 0.001
- link pelvis: geometry collision sphere radius=0.25; visual cylinder length=0.04 radius=0.015
- link r_ankle: geometry visual cylinder length=0.04 radius=0.015; visual mesh filename=../meshes/full_build_STL/Legs_Ankle_CrossGimbal2.stl scale=0.001 0.001 0.001
- link r_foot: geometry collision box size=0.2 0.10 0.03; visual cylinder length=0.04 radius=0.015
- link r_glute: geometry visual cylinder length=0.04 radius=0.015; visual mesh filename=../meshes/full_build_STL/Thigh_Right_Top_Bracket.stl scale=0.001 0.001 0.001
- link r_hipgimbal: geometry visual cylinder length=0.04 radius=0.015; visual mesh filename=../meshes/full_build_STL/Cross_Gimble.stl scale=0.001 0.001 0.001
- link r_shin: geometry visual cylinder length=0.04 radius=0.015; visual mesh filename=../meshes/full_build_STL/Right_Shin_Assembly.stl scale=0.001 0.001 0.001
- link r_thigh: geometry visual cylinder length=0.04 radius=0.015; visual mesh filename=../meshes/full_build_STL/Thigh_Right_Assembly.stl scale=0.001 0.001 0.001

Commit message: fixed feet contact and updated starting vertical position

File: resources/robots/pandora/urdf/pandora_v1_robot.urdf (robot description, URDF)
Before this commit: robot pandora_v1, 13 links, 12 joints
Links:
- link l_foot: geometry collision box size=0.03 0.10 0.2; visual box size=0.03 0.10 0.2
- link r_foot: geometry collision box size=0.03 0.10 0.2; visual box size=0.03 0.10 0.2

Commit message: made pandora top heavy and played with rewards,
need to make it more top heavy and try more time after that play with rewards again

File: resources/robots/pandora/urdf/pandora_v1_robot.urdf (robot description, URDF)
Before this commit: robot pandora_v1, 13 links, 12 joints
Links:
- link pelvis: mass 4.59 -> 14.59

Commit message: It F Walks!!!!

File: resources/robots/pandora/urdf/pandora_v1_robot.urdf (robot description, URDF)
Before this commit: robot pandora_v1, 13 links, 12 joints
Links:
- link pelvis: geometry collision sphere radius=0.8; visual cylinder length=0.04 radius=0.015

Commit message: fixing collision

File: resources/robots/pandora/urdf/pandora_v1_robot.urdf (robot description, URDF)
Before this commit: robot pandora_v1, 13 links, 12 joints
Links:
- link l_shin: geometry collision sphere radius=0.1; visual cylinder length=0.04 radius=0.015
- link pelvis: mass 14.59 -> 4.59; geometry collision sphere radius=0.4; visual cylinder length=0.04 radius=0.015
- link r_shin: geometry collision sphere radius=0.1; visual cylinder length=0.04 radius=0.015

Commit message: updated feet colision

File: resources/robots/pandora/urdf/pandora_v1_robot.urdf (robot description, URDF)
Before this commit: robot pandora_v1, 13 links, 12 joints
Links:
- link l_foot: geometry collision box size=0.03 0.13 0.22; visual box size=0.03 0.13 0.22
- link r_foot: geometry collision box size=0.03 0.13 0.22; visual box size=0.03 0.13 0.22

Commit message: re-added mas cuz it looks better
(maybe more tunning would be an alernative but we are stiking with this for now..

File: resources/robots/pandora/urdf/pandora_v1_robot.urdf (robot description, URDF)
Before this commit: robot pandora_v1, 13 links, 12 joints
Links:
- link pelvis: mass 4.59 -> 14.59; geometry collision sphere radius=0.4; visual cylinder length=0.04 radius=0.015

Commit message: Remove collision mesh visuals (Isaac Gym renderer has this built-in)

File: resources/robots/pandora/urdf/pandora_v1_robot.urdf (robot description, URDF)
Before this commit: robot pandora_v1, 13 links, 12 joints
Links:
- link l_ankle: geometry visual mesh filename=../meshes/full_build_STL/Legs_Ankle_CrossGimbal2.stl scale=0.001 0.001 0.001
- link l_foot: geometry collision box size=0.03 0.13 0.22; visual mesh filename=../meshes/full_build_STL/Left_Foot_Assembly.stl scale=0.001 0.001 0.001
- link l_glute: geometry visual mesh filename=../meshes/full_build_STL/Thigh_Top_Left_Ass.stl scale=0.001 0.001 0.001
- link l_hipgimbal: geometry visual mesh filename=../meshes/full_build_STL/Cross_Gimble.stl scale=0.001 0.001 0.001
- link l_shin: geometry visual mesh filename=../meshes/full_build_STL/Left_Shin_Assembly.stl scale=0.001 0.001 0.001
- link l_thigh: geometry visual mesh filename=../meshes/full_build_STL/Thigh_Left_Assembly.stl scale=0.001 0.001 0.001
- link pelvis: geometry collision sphere radius=0.4; visual mesh filename=../meshes/full_build_STL/Hip_Assembly.stl scale=0.001 0.001 0.001
- link r_ankle: geometry visual mesh filename=../meshes/full_build_STL/Legs_Ankle_CrossGimbal2.stl scale=0.001 0.001 0.001
- link r_foot: geometry collision box size=0.03 0.13 0.22; visual mesh filename=../meshes/full_build_STL/Right_Foot_Assembly.stl scale=0.001 0.001 0.001
- link r_glute: geometry visual mesh filename=../meshes/full_build_STL/Thigh_Right_Top_Bracket.stl scale=0.001 0.001 0.001
- link r_hipgimbal: geometry visual mesh filename=../meshes/full_build_STL/Cross_Gimble.stl scale=0.001 0.001 0.001
- link r_shin: geometry visual mesh filename=../meshes/full_build_STL/Right_Shin_Assembly.stl scale=0.001 0.001 0.001
- link r_thigh: geometry visual mesh filename=../meshes/full_build_STL/Thigh_Right_Assembly.stl scale=0.001 0.001 0.001

File: resources/robots/pandora/urdf/pandora_v1_robot_colission.urdf (robot description, URDF)
Before this commit: robot pandora_v1, 13 links, 12 joints
Links:
- link l_ankle: geometry visual mesh filename=../meshes/full_build_STL/Legs_Ankle_CrossGimbal2.stl scale=0.001 0.001 0.001
- link l_foot: geometry collision box size=0.03 0.13 0.22; visual mesh filename=../meshes/full_build_STL/Left_Foot_Assembly.stl scale=0.001 0.001 0.001
- link l_glute: geometry visual mesh filename=../meshes/full_build_STL/Thigh_Top_Left_Ass.stl scale=0.001 0.001 0.001
- link l_hipgimbal: geometry visual mesh filename=../meshes/full_build_STL/Cross_Gimble.stl scale=0.001 0.001 0.001
- link l_shin: geometry collision sphere radius=0.1; visual mesh filename=../meshes/full_build_STL/Left_Shin_Assembly.stl scale=0.001 0.001 0.001
- link l_thigh: geometry visual mesh filename=../meshes/full_build_STL/Thigh_Left_Assembly.stl scale=0.001 0.001 0.001
- link pelvis: geometry collision sphere radius=0.4; visual mesh filename=../meshes/full_build_STL/Hip_Assembly.stl scale=0.001 0.001 0.001
- link r_ankle: geometry visual mesh filename=../meshes/full_build_STL/Legs_Ankle_CrossGimbal2.stl scale=0.001 0.001 0.001
- link r_foot: geometry collision box size=0.03 0.13 0.22; visual mesh filename=../meshes/full_build_STL/Right_Foot_Assembly.stl scale=0.001 0.001 0.001
- link r_glute: geometry visual mesh filename=../meshes/full_build_STL/Thigh_Right_Top_Bracket.stl scale=0.001 0.001 0.001
- link r_hipgimbal: geometry visual mesh filename=../meshes/full_build_STL/Cross_Gimble.stl scale=0.001 0.001 0.001
- link r_shin: geometry collision sphere radius=0.1; visual mesh filename=../meshes/full_build_STL/Right_Shin_Assembly.stl scale=0.001 0.001 0.001
- link r_thigh: geometry visual mesh filename=../meshes/full_build_STL/Thigh_Right_Assembly.stl scale=0.001 0.001 0.001
