Commit message: recorded website videos

File: resources/robots/pandora/urdf/pandora_v1_robot_colission.urdf (robot description, URDF)
Before this commit: robot pandora_v1, 13 links, 12 joints
Links:
- link l_shin: geometry collision sphere radius=0.1; visual cylinder length=0.04 radius=0.015
- link r_shin: geometry collision sphere radius=0.1; visual cylinder length=0.04 radius=0.015

Commit message: Increase knee torque limits

File: resources/robots/pandora/urdf/pandora_v1_robot_colission.urdf (robot description, URDF)
Before this commit: robot pandora_v1, 13 links, 12 joints
Joints:
- joint ll4_kne_pit: limit lower=-2 upper=0 effort=100 velocity=12 -> lower=-2 upper=0 effort=200 velocity=12
- joint rl4_kne_pit: limit lower=-2 upper=0 effort=100 velocity=12 -> lower=-2 upper=0 effort=200 velocity=12
